File: Hardware/edison_mezzanine_oled.sch (EAGLE design)
At the start: 25 parts, among them J1 EDISON_CONNECTOR_FULLMOUNTING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, J2 EDISON_CONNECTOR_FULLHEADER

Commit message: Removing top-side mezzanine connector
Rerouting, increasing minimum trace width to 8mil, upping via drills to
20mil.
Parts:
- removed J2: EDISON_CONNECTOR_FULLHEADER, Edison:EDISON_CONNECTOR_FULLHEADER
Connections:
- net 1.8V: no longer J2.1.8V
- net 3.3V: no longer J2.3.3V@1, J2.3.3V@2
- net FAULT: no longer J2.FAULT
- net FW_RCVR: no longer J2.FW_RCVR
- net GND: no longer J2.GND@1, J2.GND@2, J2.GND@3, J2.GND@4, J2.GND@5, J2.GND@6
- net GP109_SPI_2_CLK: no longer J2.GP109_SPI_2_CLK
- net GP110_SPI_2_FS0: no longer J2.GP110_SPI_2_FS0
- net GP111_SPI_2_FS1: no longer J2.GP111_SPI_2_FS1
- net GP114_SPI_2_RXD: no longer J2.GP114_SPI_2_RXD
- net GP115_SPI_2_TXD: no longer J2.GP115_SPI_2_TXD
- net GP128_UART_1_CTS: no longer J2.GP128_UART_1_CTS
- net GP129_UART_1_RTS: no longer J2.GP129_UART_1_RTS
- net GP12_PWM0: no longer J2.GP12_PWM0
- net GP130_UART_1_RX: no longer J2.GP130_UART_1_RX
- net GP131_UART_1_TX: no longer J2.GP131_UART_1_TX
- net GP134_UART_2_RX: no longer J2.GP134_UART_2_RX
- net GP135_UART_2_TX: no longer J2.GP135_UART_2_TX
- net GP13_PWM1: no longer J2.GP13_PWM1
- net GP14: now also OLED1.D/!C!; no longer J2.GP14, OLED1.!RESET!
- net GP15: now also OLED1.!RESET!; no longer J2.GP15, OLED1.D/!C!
- net GP165: no longer J2.GP165
- net GP182_PWM2: no longer J2.GP182_PWM2
- net GP183_PWM3: no longer J2.GP183_PWM3
- net GP19_I2C_1_SCL: no longer J2.GP19_I2C_1_SCL
- net GP20_I2C_1_SDA: no longer J2.GP20_I2C_1_SDA
- net GP27_I2C_6_SCL: no longer J2.GP27_I2C_6_SCL
- net GP28_I2C_6_SDA: no longer J2.GP28_I2C_6_SDA
- net GP40_I2S_2_CLK: no longer J2.GP40_I2S_2_CLK
- net GP41_I2S_2_FS: no longer J2.GP41_I2S_2_FS
- net GP42_I2S_2_RXD: no longer J2.GP42_I2S_2_RXD
- net GP43_I2S_2_TXD: no longer J2.GP43_I2S_2_TXD
- net GP44: no longer J2.GP44
- net GP45: no longer J2.GP45
- net GP46: no longer J2.GP46
- net GP47: no longer J2.GP47
- net GP48: no longer J2.GP48
- net GP49: no longer J2.GP49
- net GP77_SD_0_CD#: no longer J2.GP77_SD_0_CD#
- net GP78_SD_0_CLK: no longer J2.GP78_SD_0_CLK
- net GP79_SD_0_CMD: no longer J2.GP79_SD_0_CMD
- net GP80_SD_0_DAT0: no longer J2.GP80_SD_0_DAT0
- net GP81_SD_0_DAT1: no longer J2.GP81_SD_0_DAT1
- net GP82_SD_0_DAT2: no longer J2.GP82_SD_0_DAT2
- net GP83_SD_0_DAT3: no longer J2.GP83_SD_0_DAT3
- net GP84_SD_CLK_FB: no longer J2.GP84_SD_CLK_FB
- net MSIC_SLP_CLK: no longer J2.MSIC_SLP_CLK
- net OSC_CLK_OUT: no longer J2.OSC_CLK_OUT_0
- net PSW: no longer J2.PSW
- net PWRBTN#: no longer J2.PWRBTN#
- net RCVR_MODE: no longer J2.RCVR_MODE
- net RESET_OUT#: no longer J2.RESET_OUT#
- net USB_DN: no longer J2.USB_DN
- net USB_DP: no longer J2.USB_DP
- net USB_ID: no longer J2.USB_ID
- net USB_VBUS: no longer J2.USB_VBUS
- net VSYS: no longer J2.VSYS@1, J2.VSYS@2, J2.VSYS@3
- net V_BAT_BKUP: no longer J2.V_VAT_BKUP
Other:
- note added: "EDISON"
- note removed: "BOTTOM"
- note removed: "TOP-EDISON"

Commit message: Moving screen closer towards middle of board
- Updating Edison package
- Moving Joystick and buttons towards middle of board.
Parts:
- added FID1, FID2: FIDUCIAL1X2, SparkFun-Aesthetics:FIDUCIAL1X2
Changed lines of the file:
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@@
 <part name="SJ8" library="SparkFun-Passives" deviceset="JUMPER-PAD-2-NC_BY_TRACE" device="" value=""/>
 <part name="GND10" library="SparkFun-Aesthetics" deviceset="GND" device=""/>
+<part name="FID1" library="SparkFun-Aesthetics" deviceset="FIDUCIAL" device="1X2"/>
+<part name="FID2" library="SparkFun-Aesthetics" deviceset="FIDUCIAL" device="1X2"/>
 </parts>
 <sheets>
@@
 <instance part="SJ8" gate="G$1" x="200.66" y="53.34"/>
 <instance part="GND10" gate="1" x="200.66" y="127"/>
+<instance part="FID1" gate="G$1" x="246.38" y="20.32"/>
+<instance part="FID2" gate="G$1" x="246.38" y="17.78"/>
 </instances>
 <busses>

Commit message: adding fiducials to bottom side
Parts:
- added FID3, FID4: FIDUCIAL1X2, SparkFun-Aesthetics:FIDUCIAL1X2
Changed lines of the file:
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@@
 <part name="FID1" library="SparkFun-Aesthetics" deviceset="FIDUCIAL" device="1X2"/>
 <part name="FID2" library="SparkFun-Aesthetics" deviceset="FIDUCIAL" device="1X2"/>
+<part name="FID3" library="SparkFun-Aesthetics" deviceset="FIDUCIAL" device="1X2"/>
+<part name="FID4" library="SparkFun-Aesthetics" deviceset="FIDUCIAL" device="1X2"/>
 </parts>
 <sheets>
@@
 <instance part="FID1" gate="G$1" x="246.38" y="20.32"/>
 <instance part="FID2" gate="G$1" x="246.38" y="17.78"/>
+<instance part="FID3" gate="G$1" x="243.84" y="20.32"/>
+<instance part="FID4" gate="G$1" x="243.84" y="17.78"/>
 </instances>
 <busses>
