File: Hardware/oled_block.brd (EAGLE design)
At the start: 30.5 x 44.5 mm, 29 parts, among them J1 EDISON_CONNECTOR_FULLMOUNTING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

Commit message: adding pull-up resistors to inputs. v02
Parts:
- removed LOGO1: SFE_LOGO_NAME_FLAME.1_INCH, SparkFun-Aesthetics:SFE_LOGO_NAME_FLAME_.1
- added R2, R3, R4, R5, R6, R7, R8: 10K, SparkFun-Resistors:0603-RES
- S1, S2: device SparkFun-Electromechanical:TACTILE-SWITCH-SMD -> SparkFun-Electromechanical:TACTILE_SWITCH_TALL
- moved S2 5.99 mm to (8.89, 6.35)
- moved S1 5.99 mm to (19.1, 6.35)
- turned SJ2 to 90 degrees
Connections:
- net 1.8V: now also R2.2, R3.2, R4.2, R5.2, R6.2, R7.2, R8.2
- net BUT_A: now also R7.1, S1.A2; no longer S1.1
- net BUT_B: now also R8.1, S2.A2; no longer S2.1
- net GND: now also S1.B2, S2.B2; no longer S1.3, S2.3
- net GP110_SPI_2_FS0: now also SJ2.1; no longer SJ2.3
- net GP111_SPI_2_FS1: now also SJ2.3; no longer SJ2.1
- net JOY_C: now also R6.1
- net JOY_D: now also R3.1
- net JOY_L: now also R4.1
- net JOY_R: now also R5.1
- net JOY_U: now also R2.1
Routing:
- net 1.8V: track 17.6 -> 65.1 mm
- net BUT_B: track 4.91 -> 14.0 mm
- net JOY_R: track 4.99 -> 11.3 mm
- net JOY_U: track 4.67 -> 9.72 mm
- net JOY_D: track 12.1 -> 16.6 mm
- net JOY_L: track 4.23 -> 8.46 mm
- net BUT_A: track 7.19 -> 11.3 mm
- net JOY_C: track 6.29 -> 10.1 mm
Other:
- board text added: "v02"
- board text removed: "v01"
