File: Hardware/oled_block.sch (EAGLE design)
At the start: 28 parts, among them J1 EDISON_CONNECTOR_FULLMOUNTING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

Commit message: adding pull-up resistors to inputs. v02
Parts:
- removed LOGO1: SFE_LOGO_NAME_FLAME.1_INCH, SparkFun-Aesthetics:SFE_LOGO_NAME_FLAME.1_INCH
- added R2, R3, R4, R5, R6, R7, R8: 10K, SparkFun-Resistors:10KOHM1/10W1%(0603)0603
- S1, S2: device SparkFun-Electromechanical:SWITCH-MOMENTARY-2SMD -> SparkFun-Electromechanical:SWITCH-MOMENTARY-2SMD-4
Connections:
- net 1.8V: now also R2.2, R3.2, R4.2, R5.2, R6.2, R7.2, R8.2
- net BUT_A: now also R7.1
- net BUT_B: now also R8.1
- net GP110_SPI_2_FS0: now also SJ2.1; no longer SJ2.3
- net GP111_SPI_2_FS1: now also SJ2.3; no longer SJ2.1
- net JOY_C: now also R6.1
- net JOY_D: now also R3.1
- net JOY_L: now also R4.1
- net JOY_R: now also R5.1
- net JOY_U: now also R2.1
Other:
- note added: "v02"
- note removed: "v01"
- moved on the sheet: S1, S2, S3, SJ1, SJ2, SJ3, SJ4, SJ5, SJ6, SJ7, SJ8
