File: Hardware/oled_block.sch (EAGLE design)
At the start: 34 parts, among them J1 EDISON_CONNECTOR_FULLMOUNTING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

Commit message: cleaning up some silk (v10)
Other:
- note added: "v10"
- note removed: "1.65 <= VDD <= 3.3V 3.3 <= VBAT <= 4.2V"
- note removed: "v02"
Changed lines of the file:
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@@
 <?xml version="1.0" encoding="utf-8"?>
 <!DOCTYPE eagle SYSTEM "eagle.dtd">
-<eagle version="6.5.0">
+<eagle version="7.1.0">
 <drawing>
 <settings>
@@
 <sheet>
 <plain>
-<text x="231.14" y="180.34" size="1.27" layer="97">1.65 &lt;= VDD &lt;= 3.3V
-3.3 &lt;= VBAT &lt;= 4.2V</text>
 <text x="149.86" y="7.62" size="2.54" layer="94">Jim Lindblom</text>
-<text x="238.76" y="7.62" size="2.54" layer="94">v02</text>
+<text x="238.76" y="7.62" size="2.54" layer="94">v10</text>
 </plain>
 <instances>
