File: Hardware/oled_block.sch (EAGLE design)
At the start: 34 parts, among them J1 EDISON_CONNECTOR_FULLMOUNTING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

Commit message: Ready for reds Added VSYS header No known to-do items
Parts:
- added JP1: M02PTH, SparkFun-Connectors:M02PTH
Connections:
- net GND: now also JP1.1
- net VSYS: now also JP1.2
Changed lines of the file:
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@@
 <?xml version="1.0" encoding="utf-8"?>
 <!DOCTYPE eagle SYSTEM "eagle.dtd">
-<eagle version="7.1.0">
+<eagle version="6.6.0">
 <drawing>
 <settings>
@@
 <layer number="254" name="cooling" color="7" fill="1" visible="yes" active="yes"/>
 </layers>
-<schematic xreflabel="%F%N/%S.%C%R" xrefpart="/%S.%C%R">
+<schematic xreflabel="%F%N/%S" xrefpart="/%S.%C%R">
 <attributes>
 </attributes>
@@
 <part name="SUPPLY8" library="SparkFun-Aesthetics" deviceset="1.8V" device=""/>
 <part name="SUPPLY9" library="SparkFun-Aesthetics" deviceset="1.8V" device=""/>
+<part name="JP1" library="SparkFun-Connectors" deviceset="M02" device="PTH"/>
+<part name="GND4" library="SparkFun-Aesthetics" deviceset="GND" device=""/>
 </parts>
 <sheets>
@@
 <instance part="SUPPLY8" gate="G$1" x="193.04" y="83.82"/>
 <instance part="SUPPLY9" gate="G$1" x="187.96" y="83.82"/>
+<instance part="JP1" gate="G$1" x="12.7" y="134.62"/>
+<instance part="GND4" gate="1" x="22.86" y="129.54"/>
 </instances>
 <busses>
@@
 <junction x="243.84" y="137.16"/>
 </segment>
+<segment>
+<pinref part="JP1" gate="G$1" pin="1"/>
+<pinref part="GND4" gate="1" pin="GND"/>
+<wire x1="20.32" y1="134.62" x2="22.86" y2="134.62" width="0.1524" layer="91"/>
+<wire x1="22.86" y1="134.62" x2="22.86" y2="132.08" width="0.1524" layer="91"/>
+</segment>
 </net>
 <net name="VCOMH" class="0">
@@
 <label x="149.86" y="172.72" size="1.27" layer="95" xref="yes"/>
 </segment>
-</net>
+<segment>
+<pinref part="JP1" gate="G$1" pin="2"/>
+<wire x1="20.32" y1="137.16" x2="22.86" y2="137.16" width="0.1524" layer="91"/>
+<wire x1="22.86" y1="137.16" x2="22.86" y2="139.7" width="0.1524" layer="91"/>
+<wire x1="22.86" y1="139.7" x2="25.4" y2="139.7" width="0.1524" layer="91"/>
+<label x="25.4" y="139.7" size="1.778" layer="95" xref="yes"/>
+</segment>
+</net>
